File: kicad/AudioInput/AudioInput/AudioInput.kicad_pcb (KiCad board)
At the start: 2 copper layers, 43.2 x 48.3 mm, 59 parts, among them J1 EXPAN2, J2 EXPAN1, J3 INT_AUDIO, K1 G6K-2, Q1 BS250, Q2 2N7000, U1 MCP4651, U2 LM324, U3 CD4052B

Commit message: board routed
Parts:
- removed C15, C16: 1uF, Capacitor_THT:C_Rect_L4.0mm_W2.5mm_P2.50mm
- removed J3: INT_AUDIO, Connector_PinHeader_2.54mm:PinHeader_1x04_P2.54mm_Vertical
- removed R28, R30: 100k, Resistor_THT:R_Axial_DIN0207_L6.3mm_D2.5mm_P2.54mm_Vertical
- removed R29, R31: 150k, Resistor_THT:R_Axial_DIN0207_L6.3mm_D2.5mm_P2.54mm_Vertical
- moved TP1 77.1 mm to (168.6, 110.2)
- moved C14 2.95 mm to (153.2, 94.8)
Connections:
- U3 pad 1: AUDIO_INT_IN_L -> unconnected-(U3-Pad1)
- U3 pad 12: AUDIO_INT_IN_R -> unconnected-(U3-Pad12)
Routing:
- net GND: track 0.00 -> 191.3 mm, vias 0 -> 12
- net 5v: track 0.00 -> 164.8 mm, vias 0 -> 6
- net 1.65v: track 0.00 -> 131.2 mm, vias 0 -> 10
- net 3v3: track 0.00 -> 102.4 mm, vias 0 -> 6
- net SDA: track 0.00 -> 56.2 mm, vias 0 -> 6
- net Net-(R18-Pad1): track 0.00 -> 43.8 mm, vias 0 -> 2
- net Net-(R3-Pad1): track 0.00 -> 43.5 mm, vias 0 -> 1
- net MIC_PWR_DIS: track 0.00 -> 43.1 mm, vias 0 -> 3
- net AUDIO_EN: track 0.00 -> 42.3 mm, vias 0 -> 4
- net Net-(R17-Pad1): track 0.00 -> 40.4 mm, vias 0 -> 3
- net Net-(C1-Pad1): track 0.00 -> 39.6 mm, vias 0 -> 1
- net SCL: track 0.00 -> 38.5 mm, vias 0 -> 3
- net Net-(C3-Pad1): track 0.00 -> 38.2 mm, vias 0 -> 1
- net Net-(R12-Pad2): track 0.00 -> 37.7 mm, vias 0 -> 1
- net AUDIO_L: track 0.00 -> 36.6 mm, vias 0 -> 1
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Other:
- board text added: "Audio input v0.1"

Commit message: board routed
Parts:
- moved TP1 2.21 mm to (166.4, 110.1)
- moved R17 0.24 mm to (169.4, 103.2)
- moved R2 0.20 mm to (167.3, 106.3)
- moved R8 0.13 mm to (148.0, 69.8)
- moved R18 0.11 mm to (167.2, 100.1)
- moved R3 0.10 mm to (162.1, 106.2)
- moved R16 0.07 mm to (162.1, 103.1)
Routing:
- net GND: track 191.3 -> 190.1 mm, vias 12 -> 10
- net 1.65v: track 131.2 -> 132.2 mm, vias 10 -> 9
- net SDA: track 56.2 -> 55.5 mm
Other:
- board text added: "Audio input for ZC95 v0.1"
- board text added: "^"
- board text added: "^ OPT"
- board text removed: "Audio input v0.1"
