File: kicad/OutputBoard/output.sch (KiCad schematic (older format))
At the start: 117 parts, among them J1 MAIN_BOARD_IO, J2 MAIN_BOARD_POWER, J3 MAIN_BOARD_FP, J4 Serial (3v3), Q1 AO3400A, Q10 AO3400A, Q11 IRF9Z24NPBF, Q12 AO3400A, Q2 IRF9Z24NPBF, Q3 AO3400A, Q4 AO3400A, Q5 IRF9Z24NPBF, Q6 AO3400A, Q7 AO3400A, Q8 IRF9Z24NPBF, Q9 AO3400A, U1 LM324, U2 MCP4728, U3 TPS5430DDA, U4 Pico, U5 XC6206P332MR

Commit message: Output board bom update (#23)
* update 100k resistors to be C149504 instead of C17407 (discontinued)

* update inductor from C237915 (out of stock) to C177243

* fix rotation on U2 and U3
Parts:
- L1: LCSC C237915 -> C177243
- R10, R12, R13, R15, R16, R19, R2, R21, R23, R24, R25, R27, R29, R30, R33, R35, R37, R38, R4, R40, R41, R44, R46, R48, R5, R52, R8: LCSC C17407 -> C149504
Changed lines of the file:
@@
 F 2 "Resistor_SMD:R_0805_2012Metric_Pad1.15x1.40mm_HandSolder" H 4100 1100 50  0001 C CNN
 F 3 "~" H 4100 1100 50  0001 C CNN
-F 4 "C17407" V 4100 1100 50  0001 C CNN "LCSC"
+F 4 "C149504" V 4100 1100 50  0001 C CNN "LCSC"
 	1    4100 1100
 	0    1    1    0
@@
 F 2 "Resistor_SMD:R_0805_2012Metric_Pad1.15x1.40mm_HandSolder" H 3800 1000 50  0001 C CNN
 F 3 "~" H 3800 1000 50  0001 C CNN
-F 4 "C17407" H 3800 1000 50  0001 C CNN "LCSC"
+F 4 "C149504" H 3800 1000 50  0001 C CNN "LCSC"
 	1    3800 1000
 	-1   0    0    1
@@
 F 2 "Resistor_SMD:R_0805_2012Metric_Pad1.15x1.40mm_HandSolder" H 2950 1450 50  0001 C CNN
 F 3 "~" H 2950 1450 50  0001 C CNN
-F 4 "C17407" V 2950 1450 50  0001 C CNN "LCSC"
+F 4 "C149504" V 2950 1450 50  0001 C CNN "LCSC"
 	1    2950 1450
 	0    -1   -1   0
@@
 F 2 "Resistor_SMD:R_0805_2012Metric_Pad1.15x1.40mm_HandSolder" H 3800 1800 50  0001 C CNN
 F 3 "~" H 3800 1800 50  0001 C CNN
-F 4 "C17407" H 3800 1800 50  0001 C CNN "LCSC"
+F 4 "C149504" H 3800 1800 50  0001 C CNN "LCSC"
 	1    3800 1800
 	-1   0    0    1
@@
 F 2 "Resistor_SMD:R_0805_2012Metric_Pad1.15x1.40mm_HandSolder" H 4800 1150 50  0001 C CNN
 F 3 "~" H 4800 1150 50  0001 C CNN
-F 4 "C17407" H 4800 1150 50  0001 C CNN "LCSC"
+F 4 "C149504" H 4800 1150 50  0001 C CNN "LCSC"
 	1    4800 1150
 	1    0    0    -1
@@
 F 2 "Resistor_SMD:R_0805_2012Metric_Pad1.15x1.40mm_HandSolder" H 4650 2200 50  0001 C CNN
 F 3 "~" H 4650 2200 50  0001 C CNN
-F 4 "C17407" V 4650 2200 50  0001 C CNN "LCSC"
+F 4 "C149504" V 4650 2200 50  0001 C CNN "LCSC"
 	1    4650 2200
 	0    1    1    0
@@
 F 2 "Resistor_SMD:R_0805_2012Metric_Pad1.15x1.40mm_HandSolder" H 4100 4750 50  0001 C CNN
 F 3 "~" H 4100 4750 50  0001 C CNN
-F 4 "C17407" V 4100 4750 50  0001 C CNN "LCSC"
+F 4 "C149504" V 4100 4750 50  0001 C CNN "LCSC"
 	1    4100 4750
 	0    1    1    0
@@
 F 2 "Resistor_SMD:R_0805_2012Metric_Pad1.15x1.40mm_HandSolder" H 3800 4650 50  0001 C CNN
 F 3 "~" H 3800 4650 50  0001 C CNN
-F 4 "C17407" H 3800 4650 50  0001 C CNN "LCSC"
+F 4 "C149504" H 3800 4650 50  0001 C CNN "LCSC"
 	1    3800 4650
 	-1   0    0    1
@@
 F 2 "Resistor_SMD:R_0805_2012Metric_Pad1.15x1.40mm_HandSolder" H 2950 5100 50  0001 C CNN
 F 3 "~" H 2950 5100 50  0001 C CNN
-F 4 "C17407" V 2950 5100 50  0001 C CNN "LCSC"
+F 4 "C149504" V 2950 5100 50  0001 C CNN "LCSC"
 	1    2950 5100
 	0    -1   -1   0
@@
 F 2 "Resistor_SMD:R_0805_2012Metric_Pad1.15x1.40mm_HandSolder" H 3800 5450 50  0001 C CNN
 F 3 "~" H 3800 5450 50  0001 C CNN
-F 4 "C17407" H 3800 5450 50  0001 C CNN "LCSC"
+F 4 "C149504" H 3800 5450 50  0001 C CNN "LCSC"
 	1    3800 5450
 	-1   0    0    1
@@
 F 2 "Resistor_SMD:R_0805_2012Metric_Pad1.15x1.40mm_HandSolder" H 4800 4800 50  0001 C CNN
 F 3 "~" H 4800 4800 50  0001 C CNN
-F 4 "C17407" H 4800 4800 50  0001 C CNN "LCSC"
+F 4 "C149504" H 4800 4800 50  0001 C CNN "LCSC"
 	1    4800 4800
 	1    0    0    -1
@@
 F 2 "Resistor_SMD:R_0805_2012Metric_Pad1.15x1.40mm_HandSolder" H 4650 5850 50  0001 C CNN
 F 3 "~" H 4650 5850 50  0001 C CNN
-F 4 "C17407" V 4650 5850 50  0001 C CNN "LCSC"
+F 4 "C149504" V 4650 5850 50  0001 C CNN "LCSC"
 	1    4650 5850
 	0    1    1    0
@@
 F 2 "Resistor_SMD:R_0805_2012Metric_Pad1.15x1.40mm_HandSolder" H 4100 6450 50  0001 C CNN
 F 3 "~" H 4100 6450 50  0001 C CNN
-F 4 "C17407" V 4100 6450 50  0001 C CNN "LCSC"
+F 4 "C149504" V 4100 6450 50  0001 C CNN "LCSC"
 	1    4100 6450
 	0    1    1    0
@@
 F 2 "Resistor_SMD:R_0805_2012Metric_Pad1.15x1.40mm_HandSolder" H 3800 6350 50  0001 C CNN
 F 3 "~" H 3800 6350 50  0001 C CNN
-F 4 "C17407" H 3800 6350 50  0001 C CNN "LCSC"
+F 4 "C149504" H 3800 6350 50  0001 C CNN "LCSC"
 	1    3800 6350
 	-1   0    0    1
@@
 F 2 "Resistor_SMD:R_0805_2012Metric_Pad1.15x1.40mm_HandSolder" H 2950 6800 50  0001 C CNN
 F 3 "~" H 2950 6800 50  0001 C CNN
-F 4 "C17407" V 2950 6800 50  0001 C CNN "LCSC"
+F 4 "C149504" V 2950 6800 50  0001 C CNN "LCSC"
 	1    2950 6800
 	0    -1   -1   0
@@
 F 2 "Resistor_SMD:R_0805_2012Metric_Pad1.15x1.40mm_HandSolder" H 3800 7150 50  0001 C CNN
 F 3 "~" H 3800 7150 50  0001 C CNN
-F 4 "C17407" H 3800 7150 50  0001 C CNN "LCSC"
+F 4 "C149504" H 3800 7150 50  0001 C CNN "LCSC"
 	1    3800 7150
 	-1   0    0    1
@@
 F 2 "Resistor_SMD:R_0805_2012Metric_Pad1.15x1.40mm_HandSolder" H 4800 6500 50  0001 C CNN
 F 3 "~" H 4800 6500 50  0001 C CNN
-F 4 "C17407" H 4800 6500 50  0001 C CNN "LCSC"
+F 4 "C149504" H 4800 6500 50  0001 C CNN "LCSC"
 	1    4800 6500
 	1    0    0    -1
@@
 F 2 "Resistor_SMD:R_0805_2012Metric_Pad1.15x1.40mm_HandSolder" H 4650 7550 50  0001 C CNN
 F 3 "~" H 4650 7550 50  0001 C CNN
-F 4 "C17407" V 4650 7550 50  0001 C CNN "LCSC"
+F 4 "C149504" V 4650 7550 50  0001 C CNN "LCSC"
 	1    4650 7550
 	0    1    1    0
@@
 F 2 "Resistor_SMD:R_0805_2012Metric_Pad1.15x1.40mm_HandSolder" H 4200 8450 50  0001 C CNN
 F 3 "~" H 4200 8450 50  0001 C CNN
-F 4 "C17407" H 4200 8450 50  0001 C CNN "LCSC"
+F 4 "C149504" H 4200 8450 50  0001 C CNN "LCSC"
 	1    4200 8450
 	1    0    0    -1
@@
 F 2 "Inductor_SMD:L_7.3x7.3_H3.5" H 5950 7900 50  0001 C CNN
 F 3 "~" H 5950 7900 50  0001 C CNN
-F 4 "C237915" V 5950 7900 50  0001 C CNN "LCSC"
+F 4 "C177243" V 5950 7900 50  0001 C CNN "LCSC"
 	1    5950 7900
 	0    -1   -1   0
@@
 F 2 "Resistor_SMD:R_0805_2012Metric_Pad1.15x1.40mm_HandSolder" H 1750 4200 50  0001 C CNN
 F 3 "~" H 1750 4200 50  0001 C CNN
-F 4 "C17407" V 1750 4200 50  0001 C CNN "LCSC"
+F 4 "C149504" V 1750 4200 50  0001 C CNN "LCSC"
 	1    1750 4200
 	0    -1   -1   0
@@
 F 2 "Resistor_SMD:R_0805_2012Metric_Pad1.15x1.40mm_HandSolder" H 1750 4000 50  0001 C CNN
 F 3 "~" H 1750 4000 50  0001 C CNN
-F 4 "C17407" V 1750 4000 50  0001 C CNN "LCSC"
+F 4 "C149504" V 1750 4000 50  0001 C CNN "LCSC"
 	1    1750 4000
 	0    -1   -1   0
@@
 F 2 "Resistor_SMD:R_0805_2012Metric_Pad1.15x1.40mm_HandSolder" H 2950 3100 50  0001 C CNN
 F 3 "~" H 2950 3100 50  0001 C CNN
-F 4 "C17407" V 2950 3100 50  0001 C CNN "LCSC"
+F 4 "C149504" V 2950 3100 50  0001 C CNN "LCSC"
 	1    2950 3100
 	0    -1   -1   0
@@
 F 2 "Resistor_SMD:R_0805_2012Metric_Pad1.15x1.40mm_HandSolder" H 4100 2750 50  0001 C CNN
 F 3 "~" H 4100 2750 50  0001 C CNN
-F 4 "C17407" V 4100 2750 50  0001 C CNN "LCSC"
+F 4 "C149504" V 4100 2750 50  0001 C CNN "LCSC"
 	1    4100 2750
 	0    -1   -1   0
@@
 F 2 "Resistor_SMD:R_0805_2012Metric_Pad1.15x1.40mm_HandSolder" H 3800 2650 50  0001 C CNN
 F 3 "~" H 3800 2650 50  0001 C CNN
-F 4 "C17407" V 3800 2650 50  0001 C CNN "LCSC"
+F 4 "C149504" V 3800 2650 50  0001 C CNN "LCSC"
 	1    3800 2650
 	1    0    0    -1
@@
 F 2 "Resistor_SMD:R_0805_2012Metric_Pad1.15x1.40mm_HandSolder" H 3800 3450 50  0001 C CNN
 F 3 "~" H 3800 3450 50  0001 C CNN
-F 4 "C17407" V 3800 3450 50  0001 C CNN "LCSC"
+F 4 "C149504" V 3800 3450 50  0001 C CNN "LCSC"
 	1    3800 3450
 	1    0    0    -1
@@
 F 2 "Resistor_SMD:R_0805_2012Metric_Pad1.15x1.40mm_HandSolder" H 4650 3850 50  0001 C CNN
 F 3 "~" H 4650 3850 50  0001 C CNN
-F 4 "C17407" V 4650 3850 50  0001 C CNN "LCSC"
+F 4 "C149504" V 4650 3850 50  0001 C CNN "LCSC"
 	1    4650 3850
 	0    1    1    0
@@
 F 2 "Resistor_SMD:R_0805_2012Metric_Pad1.15x1.40mm_HandSolder" H 4800 2800 50  0001 C CNN
 F 3 "~" H 4800 2800 50  0001 C CNN
-F 4 "C17407" V 4800 2800 50  0001 C CNN "LCSC"
+F 4 "C149504" V 4800 2800 50  0001 C CNN "LCSC"
 	1    4800 2800
 	1    0    0    -1
