File: kicad/OutputBoard/output.kicad_sch (KiCad schematic)
At the start: 117 parts, among them J1 MAIN_BOARD_IO, J2 MAIN_BOARD_POWER, J3 MAIN_BOARD_FP, J4 Serial (3v3), Q1 AO3400A, Q10 AO3400A, Q11 IRF9Z24NPBF, Q12 AO3400A, Q2 IRF9Z24NPBF, Q3 AO3400A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

Commit message: swap components
Parts:
- C16: LCSC C250973 -> C108360
- D3, D4, D5, D6, D7: LCSC C72043 -> C2986059
Changed lines of the file:
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@@
       (effects (font (size 1.27 1.27)) hide)
     )
-    (property "LCSC" "C72043" (id 4) (at 22.86 158.75 90)
+    (property "LCSC" "C2986059" (id 4) (at 22.86 158.75 90)
       (effects (font (size 1.27 1.27)) hide)
     )
@@
       (effects (font (size 1.27 1.27)) hide)
     )
-    (property "LCSC" "C72043" (id 4) (at 26.67 158.75 90)
+    (property "LCSC" "C2986059" (id 4) (at 26.67 158.75 90)
       (effects (font (size 1.27 1.27)) hide)
     )
@@
       (effects (font (size 1.27 1.27)) hide)
     )
-    (property "LCSC" "C72043" (id 4) (at 30.48 158.75 90)
+    (property "LCSC" "C2986059" (id 4) (at 30.48 158.75 90)
       (effects (font (size 1.27 1.27)) hide)
     )
@@
       (effects (font (size 1.27 1.27)) hide)
     )
-    (property "LCSC" "C72043" (id 4) (at 34.29 158.75 90)
+    (property "LCSC" "C2986059" (id 4) (at 34.29 158.75 90)
       (effects (font (size 1.27 1.27)) hide)
     )
@@
       (effects (font (size 1.27 1.27)) hide)
     )
-    (property "LCSC" "C72043" (id 4) (at 38.1 158.75 90)
+    (property "LCSC" "C2986059" (id 4) (at 38.1 158.75 90)
       (effects (font (size 1.27 1.27)) hide)
     )
@@
       (effects (font (size 1.27 1.27)) hide)
     )
-    (property "LCSC" "C250973" (id 4) (at 99.06 203.2 0)
-      (effects (font (size 1.27 1.27)) hide)
-    )
+    (property "LCSC" "C108360" (id 4) (at 99.06 203.2 0)
+      (effects (font (size 1.27 1.27)) hide)
+    )

Commit message: update R1 and R26 of output board to be C479327 instead of C479296 (#121)
Parts:
- R1, R26: LCSC C479296 -> C479327
Changed lines of the file:
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@@
       (effects (font (size 1.27 1.27)) hide)
     )
-    (property "LCSC" "C479296" (id 4) (at 105.41 16.51 90)
+    (property "LCSC" "C479327" (id 4) (at 105.41 16.51 90)
       (effects (font (size 1.27 1.27)) hide)
     )
@@
       (effects (font (size 1.27 1.27)) hide)
     )
-    (property "LCSC" "C479296" (id 4) (at 105.41 109.22 90)
-      (effects (font (size 1.27 1.27)) hide)
-    )
+    (property "LCSC" "C479327" (id 4) (at 105.41 109.22 90)
+      (effects (font (size 1.27 1.27)) hide)
+    )
