File: kicad/FrontPanelControls/PanelControls.sch (KiCad schematic (older format))
At the start: 35 parts, among them J1 Conn_02x04_Odd_Even, SW5 ADJ, U1 PCF8591, U2 PCF8574, U3 WS2812D, U4 WS2812D, U5 WS2812D, U6 WS2812D, U7 WS2812D, U8 WS2812D

Commit message: update BoM and build notes (#39)
- Update 10uF cap C191532 -> C88739
- Update pin socket C50984 -> C124410
- Add comment about orientation of PCF8591 to build notes
Parts:
- C2, C4: LCSC C191532 -> C88739
Changed lines of the file:
@@
 F 2 "Capacitor_THT:CP_Radial_D4.0mm_P2.00mm" H 4490 1025 50  0001 C CNN
 F 3 "~" H 4490 1025 50  0001 C CNN
-F 4 "C191532" H 4490 1025 50  0001 C CNN "LCSC"
+F 4 "C88739" H 4490 1025 50  0001 C CNN "LCSC"
 	1    4490 1025
 	1    0    0    -1
@@
 F 2 "Capacitor_THT:CP_Radial_D4.0mm_P1.50mm" H 4940 1825 50  0001 C CNN
 F 3 "~" H 4940 1825 50  0001 C CNN
-F 4 "C191532" H 4940 1825 50  0001 C CNN "LCSC"
+F 4 "C88739" H 4940 1825 50  0001 C CNN "LCSC"
 	1    4940 1825
 	1    0    0    -1
