File: kicad/MainBoard/MainBoard.kicad_pcb (KiCad board)
At the start: 2 copper layers, 191.5 x 166.3 mm, 104 parts, among them J1 CHAN1, J10 ACC Port, J11 433TX, J12 VDC INPUT, J13 BAT, J14 TRG1, J15 TRG2, J16 FP-BUTTONS, J17 EXPAN2, J18 OUTPUT_BOARD_POWER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

Commit message: fix board outline for front panel and mainboad (#139)
Other:
- net class Default removed
