File: kicad/MainBoard/main.kicad_pcb (KiCad board)
At the start: 2 copper layers, 191.5 x 76 mm, 323 parts, among them J1 TRG1, J10 I2C, J11 CHAN1, J12 CHAN2, J13 Conn_01x02, J14 CHAN3, J15 CHAN4, J16 Conn_01x02_Female, J18 AudioJack3_SwitchTR, J2 TRG2, J20 USB_C_Receptacle, J3 Conn_02x04_Odd_Even, J4 AudioJack3_SwitchTR, J5 Conn_02x04_Odd_Even, J6 LCD, J7 ACC Port, J8 FrontPanel, J9 433TX, Q1 AO3401A, Q10 AO3400A, Q11 AO3400A, Q12 IRF9Z24NPBF, Q13 AO3400A, Q14 AO3401A, Q15 AO3401A, Q16 AO3401A, Q17 AO3401A, Q18 AO3401A, Q19 AO3400A, Q2 AO3400A, Q3 IRF9Z24NPBF, Q4 AO3400A, Q5 AO3400A, Q6 IRF9Z24NPBF, Q7 AO3400A, Q8 AO3400A, Q9 IRF9Z24NPBF, SW1 Power switch, U1 TCA9534, U10 MCP4651, U11 LM324, U12 SN74LVC1G3157DCKR, U13 BQ27441-G1, U14 HY2111-GB, U15 FS8205A, U16 TP4056, U17 TPS61088, U18 SN74LVC1G3157DCKR, U19 USBLC6-2P6, U20 USBLC6-2P6, U21 USBLC6-2P6, U22 USBLC6-2P6, U23 USBLC6-2P6, U24 USBLC6-2P6, U25 USBLC6-2P6, U28 TCA9534, U3 Pico, U4 MAX3232EEAE+T, U5 AT24C04CDRG, U6 LM324, U7 MCP4728, U8 TPS61088, U9 Pico

Commit message: fix solder mask minimum width setting, then regenerate gerbers
Other:
- board text added: "ZC95 Mark II v2.1 - CrashOverride85"
- board text removed: "ZC95 Mark II v2.0 - CrashOverride85"
Changed lines of the file:
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@@
     )
     (pad_to_mask_clearance 0.051)
-    (solder_mask_min_width 0.25)
     (pcbplotparams
       (layerselection 0x00010fc_ffffffff)
@@
     (effects (font (size 2 2) (thickness 0.3)))
   )
-  (gr_text "ZC95 Mark II v2.0 - CrashOverride85" (at 189.56 59.36) (layer "F.SilkS")
+  (gr_text "ZC95 Mark II v2.1 - CrashOverride85" (at 189.56 59.36) (layer "F.SilkS")
     (effects (font (size 1.5 1.5) (thickness 0.3)))
   )
