File: kicad/MainBoard/main.kicad_pcb (KiCad board)
At the start: 2 copper layers, 191.5 x 76 mm, 331 parts, among them J1 TRG1, J10 I2C, J11 CHAN1, J12 CHAN2, J13 Conn_01x02, J14 CHAN3, J15 CHAN4, J16 Conn_01x02_Female, J18 AudioJack3_SwitchTR, J2 TRG2, J20 USB_C_Receptacle, J3 Conn_02x04_Odd_Even, J4 AudioJack3_SwitchTR, J5 Conn_02x04_Odd_Even, J6 LCD, J7 ACC Port, J8 FrontPanel, J9 433TX, Q1 AO3401A, Q10 AO3400A, Q11 AO3400A, Q12 IRF9Z24NPBF, Q13 AO3400A, Q14 AO3401A, Q15 AO3401A, Q18 AO3401A, Q19 AO3400A, Q2 AO3400A, Q3 IRF9Z24NPBF, Q4 AO3400A, Q5 AO3400A, Q6 IRF9Z24NPBF, Q7 AO3400A, Q8 AO3400A, Q9 IRF9Z24NPBF, SW1 SW_SPDT, U1 TCA9534, U10 MCP4651, U11 LM324, U12 SN74LVC1G3157DCKR, U13 BQ27441-G1, U14 HY2111-GB, U15 FS8205A, U16 HT7533-1, U17 TPS61088, U18 SN74LVC1G3157DCKR, U19 USBLC6-2P6, U2 BQ25601, U20 USBLC6-2P6, U21 USBLC6-2P6, U22 USBLC6-2P6, U23 USBLC6-2P6, U24 USBLC6-2P6, U25 USBLC6-2P6, U26 SN74LVC1G3157DCKR, U27 SN74LVC1G3157DCKR, U28 TCA9534, U3 Pico, U4 MAX3232EEAE+T, U5 AT24C04CDRG, U6 LM324, U7 MCP4728, U8 TPS61088, U9 Pico

Commit message: v2.5 schematic + PCB changes
Parts:
- added Q16: AO3401A, Package_TO_SOT_SMD:SOT-23_Handsoldering, F.Cu at (149.6, 100.8)
- added Q17: AO3400A, Package_TO_SOT_SMD:SOT-23_Handsoldering, F.Cu at (155.1, 94.5)
- added R155: 10k, Resistor_SMD:R_0603_1608Metric_Pad0.98x0.95mm_HandSolder, F.Cu at (155.7, 99.2)
Connections:
- C52 pad 2: 5v -> Net-(C52-Pad2)
- C53 pad 1: 5v -> Net-(C52-Pad2)
- C54 pad 1: 5v -> Net-(C52-Pad2)
- C55 pad 1: 5v -> Net-(C52-Pad2)
- R141 pad 2: 5v -> Net-(C52-Pad2)
- R142 pad 1: 5v -> Net-(C52-Pad2)
- TP3 pad 1: 5v -> Net-(C52-Pad2)
- U17 pad 14: 5v -> Net-(C52-Pad2)
- U17 pad 15: 5v -> Net-(C52-Pad2)
- U17 pad 16: 5v -> Net-(C52-Pad2)
Routing:
- net Net-(C52-Pad2): track 0.00 -> 13.4 mm
- net 5v: track 423.3 -> 410.1 mm, vias 26 -> 27
- net PWR_EN: track 228.5 -> 239.5 mm
- net Net-(Q16-Pad1): track 0.00 -> 8.36 mm
- net GND: vias 392 -> 398
- added copper zone on F.Cu, net Net-(C52-Pad2)
- removed copper zone on F.Cu, net 5v
Other:
- board text added: "ZC95 Mark II v2.5 - CrashOverride85"
- board text removed: "ZC95 Mark II v2.4 - CrashOverride85"

Commit message: tweaks
Parts:
- moved R37 1.05 mm to (232.3, 82.0)
Routing:
- net 5v: track 410.1 -> 409.5 mm
