File: kicad/MainBoard/main.kicad_pcb (KiCad board)
At the start: 2 copper layers, 191.5 x 76 mm, 334 parts, among them J1 TRG1, J10 I2C, J11 CHAN1, J12 CHAN2, J13 Conn_01x02, J14 CHAN3, J15 CHAN4, J16 Conn_01x02_Female, J18 AudioJack3_SwitchTR, J2 TRG2, J20 USB_C_Receptacle, J3 Conn_02x04_Odd_Even, J4 AudioJack3_SwitchTR, J5 Conn_02x04_Odd_Even, J6 LCD, J7 ACC Port, J8 FrontPanel, J9 433TX, Q1 AO3401A, Q10 AO3400A, Q11 AO3400A, Q12 IRF9Z24NPBF, Q13 AO3400A, Q14 AO3401A, Q15 AO3401A, Q16 AO3401A, Q17 AO3400A, Q18 AO3401A, Q19 AO3400A, Q2 AO3400A, Q3 IRF9Z24NPBF, Q4 AO3400A, Q5 AO3400A, Q6 IRF9Z24NPBF, Q7 AO3400A, Q8 AO3400A, Q9 IRF9Z24NPBF, SW1 SW_SPDT, U1 TCA9534, U10 MCP4651, U11 LM324, U12 SN74LVC1G3157DCKR, U13 BQ27441-G1, U14 HY2111-GB, U15 FS8205A, U16 HT7533-1, U17 TPS61088, U18 SN74LVC1G3157DCKR, U19 USBLC6-2P6, U2 BQ25601, U20 USBLC6-2P6, U21 USBLC6-2P6, U22 USBLC6-2P6, U23 USBLC6-2P6, U24 USBLC6-2P6, U25 USBLC6-2P6, U26 SN74LVC1G3157DCKR, U27 SN74LVC1G3157DCKR, U28 TCA9534, U3 Pico, U4 MAX3232EEAE+T, U5 AT24C04CDRG, U6 LM324, U7 MCP4728, U8 TPS61088, U9 Pico

Commit message: Change C50 on main board from 4.7nF to 47nF
Parts:
- C50: value 4.7nF -> 47nF
Changed lines of the file:
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@@
     (descr "Capacitor SMD 0603 (1608 Metric), square (rectangular) end terminal, IPC_7351 nominal with elongated pad for handsoldering. (Body size source: IPC-SM-782 page 76, https://www.pcb-3d.com/wordpress/wp-content/uploads/ipc-sm-782a_amendment_1_and_2.pdf), generated with kicad-footprint-generator")
     (tags "capacitor handsolder")
-    (property "LCSC" "C53987")
+    (property "LCSC" "C1622")
     (property "Sheetfile" "power.kicad_sch")
     (property "Sheetname" "Power")
@@
       (effects (font (size 0.7 0.7) (thickness 0.15)))
     )
-    (fp_text value "4.7nF" (at 0 1.43) (layer "F.Fab")
+    (fp_text value "47nF" (at 0 1.43) (layer "F.Fab")
       (effects (font (size 1 1) (thickness 0.15)))
     )

Commit message: C58 on the mainboard should be 10uF not 10nF
Parts:
- C58: value 10nF -> 10uF
Changed lines of the file:
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@@
     (descr "Capacitor SMD 0603 (1608 Metric), square (rectangular) end terminal, IPC_7351 nominal with elongated pad for handsoldering. (Body size source: IPC-SM-782 page 76, https://www.pcb-3d.com/wordpress/wp-content/uploads/ipc-sm-782a_amendment_1_and_2.pdf), generated with kicad-footprint-generator")
     (tags "capacitor handsolder")
-    (property "LCSC" "C57112")
+    (property "LCSC" "C19702")
     (property "Sheetfile" "power.kicad_sch")
     (property "Sheetname" "Power")
@@
       (effects (font (size 0.7 0.7) (thickness 0.15)))
     )
-    (fp_text value "10nF" (at 0 1.43) (layer "F.Fab")
+    (fp_text value "10uF" (at 0 1.43) (layer "F.Fab")
       (effects (font (size 1 1) (thickness 0.15)))
     )
