File: kicad/MainBoard/audio.kicad_sch (KiCad schematic)
At the start: 53 parts, among them J18 AudioJack3_SwitchTR, Q14 AO3401A, Q15 AO3401A, U10 MCP4651, U11 LM324, U12 SN74LVC1G3157DCKR, U16 HT7533-1, U18 SN74LVC1G3157DCKR, U25 USBLC6-2P6

Commit message: Pcb v2.6 (#167)
Parts:
- added J16: AudioIn, Connector_PinSocket_2.54mm:PinSocket_1x03_P2.54mm_Vertical, symbol Connector_Generic:Conn_01x03
Connections:
- net GND: now also J16.2 (Pin_2)
- net at J18.RN: now also J16.3 (Pin_3)
- net at J18.TN: now also J16.1 (Pin_1)
- no-connect marks 4 -> 2
Other:
- moved on the sheet: C32, C36, D28, J18, Q14, Q15, R116, R120, R121, R123, R124, U25
